File: BuitPCB/Sensors.sch (KiCad schematic (older format))
At the start: 3 parts, among them J5 LEFT SENS, J7 RIGHT SENS, J9 CENTER SENS

Commit message: Updated to almost every component and started routing
Parts:
- J5: value LEFT SENS -> LEFT VL
- J7: value RIGHT SENS -> RIGHT VL
- J9: value CENTER SENS -> CENTER VL
Changed lines of the file:
@@
 P 4100 3600
 F 0 "J5" H 4180 3642 50  0000 L CNN
-F 1 "LEFT SENS" H 4180 3551 50  0000 L CNN
+F 1 "LEFT VL" H 4180 3551 50  0000 L CNN
 F 2 "Connector_JST:JST_XH_B5B-XH-A_1x05_P2.50mm_Vertical" H 4100 3600 50  0001 C CNN
 F 3 "~" H 4100 3600 50  0001 C CNN
@@
 P 6300 3600
 F 0 "J7" H 6380 3642 50  0000 L CNN
-F 1 "RIGHT SENS" H 6380 3551 50  0000 L CNN
+F 1 "RIGHT VL" H 6380 3551 50  0000 L CNN
 F 2 "Connector_JST:JST_XH_B5B-XH-A_1x05_P2.50mm_Vertical" H 6300 3600 50  0001 C CNN
 F 3 "~" H 6300 3600 50  0001 C CNN
@@
 P 8500 3600
 F 0 "J9" H 8580 3642 50  0000 L CNN
-F 1 "CENTER SENS" H 8580 3551 50  0000 L CNN
+F 1 "CENTER VL" H 8580 3551 50  0000 L CNN
 F 2 "Connector_JST:JST_XH_B5B-XH-A_1x05_P2.50mm_Vertical" H 8500 3600 50  0001 C CNN
 F 3 "~" H 8500 3600 50  0001 C CNN
