File: BuitPCB/DevBoard.kicad_sch (KiCad schematic)
At the start: 2 parts, among them U1 Teensy4.1, U6 ESP8266

Commit message: Updated almost to final 0.1 version
Parts:
- added C12, C5, C6: 100nF, Capacitor_SMD:C_0805_2012Metric, symbol Device:C
Connections:
- net +3V3: now also U1.46 (3V3)
- net GND: now also C12.1, C5.1, C6.1
- net ROT_CLICK_SW: now reaches U1.12 (10_CS_MQSR)
- net ROT_CLICK_DT: now reaches U1.13 (11_MOSI_CTX1)
- net ROT_CLICK_CLK: now reaches U1.14 (12_MISO_MQSL)
- net +5V: now reaches U1.48 (VIN)
- net +5V: now also C12.2, C5.2, C6.2
- net USB_HOST_D+ renamed USB_HOST_P
- net USB_HOST_D- renamed USB_HOST_N
- net V_USB: no longer names the net of U1.49 (VUSB)
Changed lines of the file:
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@@
 (kicad_sch (version 20211123) (generator eeschema)
   (paper "A4")
+  (junction (at 199.39 38.1) (diameter 0) (color 0 0 0 0)
+  )
+  (junction (at 212.09 38.1) (diameter 0) (color 0 0 0 0)
+  )
+  (junction (at 186.69 38.1) (diameter 0) (color 0 0 0 0)
+  )
   (junction (at 193.04 76.2) (diameter 0) (color 0 0 0 0)
   )
+  (wire (pts (xy 186.69 38.1) (xy 199.39 38.1))
+    (stroke (width 0) (type default) (color 0 0 0 0))
+  )
+  (wire (pts (xy 181.61 38.1) (xy 186.69 38.1))
+    (stroke (width 0) (type default) (color 0 0 0 0))
+  )
+  (wire (pts (xy 218.44 36.83) (xy 218.44 38.1))
+    (stroke (width 0) (type default) (color 0 0 0 0))
+  )
+  (wire (pts (xy 199.39 38.1) (xy 212.09 38.1))
+    (stroke (width 0) (type default) (color 0 0 0 0))
+  )
   (wire (pts (xy 194.31 76.2) (xy 193.04 76.2))
     (stroke (width 0) (type default) (color 0 0 0 0))
@@
     (stroke (width 0) (type default) (color 0 0 0 0))
   )
+  (wire (pts (xy 212.09 38.1) (xy 218.44 38.1))
+    (stroke (width 0) (type default) (color 0 0 0 0))
+  )
   (global_label "I2S_DIN" (shape input) (at 66.04 64.77 180) (fields_autoplaced)
     (effects (font (size 1.27 1.27)) (justify right))
@@
     )
   )
+  (global_label "ROT_CLICK_SW" (shape input) (at 66.04 72.39 180) (fields_autoplaced)
+    (effects (font (size 1.27 1.27)) (justify right))
+    (property "Intersheet References" "${INTERSHEET_REFS}" (id 0) (at 50.1087 72.3106 0)
+      (effects (font (size 1.27 1.27)) (justify right) hide)
+    )
+  )
+  (global_label "V_USB" (shape input) (at 181.61 38.1 180) (fields_autoplaced)
+    (effects (font (size 1.27 1.27)) (justify right))
+    (property "Intersheet References" "${INTERSHEET_REFS}" (id 0) (at 303.53 78.74 0)
+      (effects (font (size 1.27 1.27)) hide)
+    )
+  )
   (global_label "ESP8266_UART_RX" (shape input) (at 213.36 76.2 0) (fields_autoplaced)
     (effects (font (size 1.27 1.27)) (justify left))
@@
     )
   )
+  (global_label "ROT_CLICK_CLK" (shape input) (at 66.04 77.47 180) (fields_autoplaced)
+    (effects (font (size 1.27 1.27)) (justify right))
+    (property "Intersheet References" "${INTERSHEET_REFS}" (id 0) (at 49.2015 77.3906 0)
+      (effects (font (size 1.27 1.27)) (justify right) hide)
+    )
+  )
   (global_label "USB_HOST_5V" (shape input) (at 66.04 114.3 180) (fields_autoplaced)
     (effects (font (size 1.27 1.27)) (justify right))
@@
     )
   )
-  (global_label "USB_HOST_D+" (shape input) (at 66.04 119.38 180) (fields_autoplaced)
-    (effects (font (size 1.27 1.27)) (justify right))
-    (property "Intersheet References" "${INTERSHEET_REFS}" (id 0) (at 0 0 0)
-      (effects (font (size 1.27 1.27)) hide)
+  (global_label "USB_HOST_P" (shape input) (at 66.04 119.38 180) (fields_autoplaced)
+    (effects (font (size 1.27 1.27)) (justify right))
+    (property "Intersheet References" "${INTERSHEET_REFS}" (id 0) (at 51.8625 119.3006 0)
+      (effects (font (size 1.27 1.27)) (justify right) hide)
     )
   )
@@
     )
   )
+  (global_label "ROT_CLICK_DT" (shape input) (at 66.04 74.93 180) (fields_autoplaced)
+    (effects (font (size 1.27 1.27)) (justify right))
+    (property "Intersheet References" "${INTERSHEET_REFS}" (id 0) (at 50.532 74.8506 0)
+      (effects (font (size 1.27 1.27)) (justify right) hide)
+    )
+  )
   (global_label "I2C_SDA_3V3" (shape input) (at 121.92 64.77 0) (fields_autoplaced)
     (effects (font (size 1.27 1.27)) (justify left))
@@
     )
   )
-  (global_label "V_USB" (shape input) (at 121.92 40.64 0) (fields_autoplaced)
-    (effects (font (size 1.27 1.27)) (justify left))
-    (property "Intersheet References" "${INTERSHEET_REFS}" (id 0) (at 0 0 0)
+  (global_label "V_USB" (shape input) (at 121.92 44.45 0) (fields_autoplaced)
+    (effects (font (size 1.27 1.27)) (justify left))
+    (property "Intersheet References" "${INTERSHEET_REFS}" (id 0) (at 0 3.81 0)
       (effects (font (size 1.27 1.27)) hide)
     )
@@
     )
   )
-  (global_label "USB_HOST_D-" (shape input) (at 66.04 116.84 180) (fields_autoplaced)
-    (effects (font (size 1.27 1.27)) (justify right))
-    (property "Intersheet References" "${INTERSHEET_REFS}" (id 0) (at 0 0 0)
-      (effects (font (size 1.27 1.27)) hide)
+  (global_label "USB_HOST_N" (shape input) (at 66.04 116.84 180) (fields_autoplaced)
+    (effects (font (size 1.27 1.27)) (justify right))
+    (property "Intersheet References" "${INTERSHEET_REFS}" (id 0) (at 51.802 116.7606 0)
+      (effects (font (size 1.27 1.27)) (justify right) hide)
     )
   )
@@
     )
   )
-  (symbol (lib_id "teensy:Teensy4.1") (at 93.98 99.06 0)
+  (symbol (lib_id "teensy:Teensy4.1") (at 93.98 99.06 0) (unit 1)
     (in_bom yes) (on_board yes)
     (property "Reference" "U1" (id 0) (at 93.98 33.909 0))
@@
       (effects (font (size 1.27 1.27)) hide)
     )
+    (pin "1")
+  )
+  (symbol (lib_id "power:GND") (at 199.39 45.72 0) (unit 1)
+    (in_bom yes) (on_board yes)
+    (property "Reference" "#PWR015" (id 0) (at 199.39 52.07 0)
+      (effects (font (size 1.27 1.27)) hide)
+    )
+    (property "Value" "GND" (id 1) (at 199.517 50.1142 0))
+    (property "Footprint" "" (id 2) (at 199.39 45.72 0)
+      (effects (font (size 1.27 1.27)) hide)
+    )
+    (property "Datasheet" "" (id 3) (at 199.39 45.72 0)
+      (effects (font (size 1.27 1.27)) hide)
+    )
+    (pin "1")
+  )
+  (symbol (lib_id "power:+3V3") (at 121.92 49.53 270) (unit 1)
+    (in_bom yes) (on_board yes)
+    (property "Reference" "#PWR013" (id 0) (at 118.11 49.53 0)
+      (effects (font (size 1.27 1.27)) hide)
+    )
+    (property "Value" "+3V3" (id 1) (at 125.1712 49.911 90)
+      (effects (font (size 1.27 1.27)) (justify left))
+    )
+    (property "Footprint" "" (id 2) (at 121.92 49.53 0)
+      (effects (font (size 1.27 1.27)) hide)
+    )
+    (property "Datasheet" "" (id 3) (at 121.92 49.53 0)
+      (effects (font (size 1.27 1.27)) hide)
+    )
+    (pin "1")
+  )
+  (symbol (lib_id "Device:C") (at 212.09 41.91 180) (unit 1)
+    (in_bom yes) (on_board yes)
+    (property "Reference" "C12" (id 0) (at 209.169 43.0784 0)
+      (effects (font (size 1.27 1.27)) (justify left))
+    )
+    (property "Value" "100nF" (id 1) (at 209.169 40.767 0)
+      (effects (font (size 1.27 1.27)) (justify left))
+    )
+    (property "Footprint" "Capacitor_SMD:C_0805_2012Metric" (id 2) (at 211.1248 38.1 0)
+      (effects (font (size 1.27 1.27)) hide)
+    )
+    (property "Datasheet" "~" (id 3) (at 212.09 41.91 0)
+      (effects (font (size 1.27 1.27)) hide)
+    )
+    (pin "1")
+    (pin "2")
+  )
+  (symbol (lib_id "Device:C") (at 199.39 41.91 180) (unit 1)
+    (in_bom yes) (on_board yes)
+    (property "Reference" "C6" (id 0) (at 196.469 43.0784 0)
+      (effects (font (size 1.27 1.27)) (justify left))
+    )
+    (property "Value" "100nF" (id 1) (at 196.469 40.767 0)
+      (effects (font (size 1.27 1.27)) (justify left))
+    )
+    (property "Footprint" "Capacitor_SMD:C_0805_2012Metric" (id 2) (at 198.4248 38.1 0)
+      (effects (font (size 1.27 1.27)) hide)
+    )
+    (property "Datasheet" "~" (id 3) (at 199.39 41.91 0)
+      (effects (font (size 1.27 1.27)) hide)
+    )
+    (pin "1")
+    (pin "2")
+  )
+  (symbol (lib_id "Device:C") (at 186.69 41.91 180) (unit 1)
+    (in_bom yes) (on_board yes)
+    (property "Reference" "C5" (id 0) (at 183.769 43.0784 0)
+      (effects (font (size 1.27 1.27)) (justify left))
+    )
+    (property "Value" "100nF" (id 1) (at 183.769 40.767 0)
+      (effects (font (size 1.27 1.27)) (justify left))
+    )
+    (property "Footprint" "Capacitor_SMD:C_0805_2012Metric" (id 2) (at 185.7248 38.1 0)
+      (effects (font (size 1.27 1.27)) hide)
+    )
+    (property "Datasheet" "~" (id 3) (at 186.69 41.91 0)
+      (effects (font (size 1.27 1.27)) hide)
+    )
+    (pin "1")
+    (pin "2")
+  )
+  (symbol (lib_id "power:GND") (at 212.09 45.72 0) (unit 1)
+    (in_bom yes) (on_board yes)
+    (property "Reference" "#PWR020" (id 0) (at 212.09 52.07 0)
+      (effects (font (size 1.27 1.27)) hide)
+    )
+    (property "Value" "GND" (id 1) (at 212.217 50.1142 0))
+    (property "Footprint" "" (id 2) (at 212.09 45.72 0)
+      (effects (font (size 1.27 1.27)) hide)
+    )
+    (property "Datasheet" "" (id 3) (at 212.09 45.72 0)
+      (effects (font (size 1.27 1.27)) hide)
+    )
+    (pin "1")
+  )
+  (symbol (lib_id "power:GND") (at 186.69 45.72 0) (unit 1)
+    (in_bom yes) (on_board yes)
+    (property "Reference" "#PWR014" (id 0) (at 186.69 52.07 0)
+      (effects (font (size 1.27 1.27)) hide)
+    )
+    (property "Value" "GND" (id 1) (at 186.817 50.1142 0))
+    (property "Footprint" "" (id 2) (at 186.69 45.72 0)
+      (effects (font (size 1.27 1.27)) hide)
+    )
+    (property "Datasheet" "" (id 3) (at 186.69 45.72 0)
+      (effects (font (size 1.27 1.27)) hide)
+    )
+    (pin "1")
+  )
+  (symbol (lib_id "power:+5V") (at 218.44 36.83 0) (unit 1)
+    (in_bom yes) (on_board yes) (fields_autoplaced)
+    (property "Reference" "#PWR021" (id 0) (at 218.44 40.64 0)
+      (effects (font (size 1.27 1.27)) hide)
+    )
+    (property "Value" "+5V" (id 1) (at 218.44 33.2255 0))
+    (property "Footprint" "" (id 2) (at 218.44 36.83 0)
+      (effects (font (size 1.27 1.27)) hide)
+    )
+    (property "Datasheet" "" (id 3) (at 218.44 36.83 0)
+      (effects (font (size 1.27 1.27)) hide)
+    )
