File: BuitPCB/i2cBu&Conn.kicad_sch (KiCad schematic)
At the start: 2 parts, among them J11 OLED DISPLAY, J12 NEO TRELLIS

Commit message: Updated almost to final 0.1 version
Parts:
- added R5, R6: 3K3, Resistor_SMD:R_0805_2012Metric, symbol Device:R
Connections:
- net +3V3: now also R5.1, R6.1
- net I2C_SCL_3V3: now also R5.2
- net I2C_SDA_3V3: now also R6.2
Changed lines of the file:
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@@
+    )
+  )
+  (global_label "I2C_SDA_3V3" (shape input) (at 86.36 83.82 180) (fields_autoplaced)
+    (effects (font (size 1.27 1.27)) (justify right))
+    (property "Intersheet References" "${INTERSHEET_REFS}" (id 0) (at -81.28 -2.54 0)
+      (effects (font (size 1.27 1.27)) hide)
+    )
+  )
+  (global_label "I2C_SCL_3V3" (shape input) (at 86.36 71.12 180) (fields_autoplaced)
+    (effects (font (size 1.27 1.27)) (justify right))
+    (property "Intersheet References" "${INTERSHEET_REFS}" (id 0) (at -81.28 -12.7 0)
+      (effects (font (size 1.27 1.27)) hide)
     )
   )
@@
     (pin "5")
   )
+  (symbol (lib_id "power:+3V3") (at 93.98 83.82 270) (unit 1)
+    (in_bom yes) (on_board yes)
+    (property "Reference" "#PWR0117" (id 0) (at 90.17 83.82 0)
+      (effects (font (size 1.27 1.27)) hide)
+    )
+    (property "Value" "+3V3" (id 1) (at 96.52 83.82 90)
+      (effects (font (size 1.27 1.27)) (justify left))
+    )
+    (property "Footprint" "" (id 2) (at 93.98 83.82 0)
+      (effects (font (size 1.27 1.27)) hide)
+    )
+    (property "Datasheet" "" (id 3) (at 93.98 83.82 0)
+      (effects (font (size 1.27 1.27)) hide)
+    )
+    (pin "1")
+  )
+  (symbol (lib_id "power:+3V3") (at 93.98 71.12 270) (unit 1)
+    (in_bom yes) (on_board yes)
+    (property "Reference" "#PWR0116" (id 0) (at 90.17 71.12 0)
+      (effects (font (size 1.27 1.27)) hide)
+    )
+    (property "Value" "+3V3" (id 1) (at 96.52 71.12 90)
+      (effects (font (size 1.27 1.27)) (justify left))
+    )
+    (property "Footprint" "" (id 2) (at 93.98 71.12 0)
+      (effects (font (size 1.27 1.27)) hide)
+    )
+    (property "Datasheet" "" (id 3) (at 93.98 71.12 0)
+      (effects (font (size 1.27 1.27)) hide)
+    )
+    (pin "1")
+  )
+  (symbol (lib_id "Device:R") (at 90.17 71.12 270) (unit 1)
+    (in_bom yes) (on_board yes)
+    (property "Reference" "R5" (id 0) (at 90.17 65.8622 90))
+    (property "Value" "3K3" (id 1) (at 90.17 68.1736 90))
+    (property "Footprint" "Resistor_SMD:R_0805_2012Metric" (id 2) (at 90.17 69.342 90)
+      (effects (font (size 1.27 1.27)) hide)
+    )
+    (property "Datasheet" "~" (id 3) (at 90.17 71.12 0)
+      (effects (font (size 1.27 1.27)) hide)
+    )
+    (pin "1")
+    (pin "2")
+  )
+  (symbol (lib_id "Device:R") (at 90.17 83.82 270) (unit 1)
+    (in_bom yes) (on_board yes)
+    (property "Reference" "R6" (id 0) (at 90.17 78.5622 90))
+    (property "Value" "3K3" (id 1) (at 90.17 80.8736 90))
+    (property "Footprint" "Resistor_SMD:R_0805_2012Metric" (id 2) (at 90.17 82.042 90)
+      (effects (font (size 1.27 1.27)) hide)
+    )
+    (property "Datasheet" "~" (id 3) (at 90.17 83.82 0)
+      (effects (font (size 1.27 1.27)) hide)
+    )
+    (pin "1")
+    (pin "2")
+  )
 )
