File: BuitPCB/BuitPCB.kicad_pcb (KiCad board)
At the start: 4 copper layers, 100 x 100 mm, 43 parts, among them J1 MIDI IN, J10 ROTARY CLICK, J11 OLED DISPLAY, J12 NEO TRELLIS, J2 MIDI OUT, J3 USB HOST, J4 LINE IN, J5 LEFT VL, J6 HEAD/OUT, J7 RIGHT VL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

Commit message: updated with almost al 3d models and esp001 rotated
Parts:
- REF**: value TestPoint_Plated_Hole_D3.0mm -> (none)
- moved U6 15.9 mm to (122.1, 84.7), turned to 180 degrees
Routing:
- net ESP8266_UART_RX: track 56.8 -> 72.6 mm
- net ESP8266_UART_TX: track 51.1 -> 53.0 mm
Changed lines of the file:
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@@
       (net 62 "unconnected-(U1-Pad67)") (pinfunction "D+") (pintype "bidirectional"))
     (model "C:/Users/xamps/Documents/Electronics/libs/CIRCUIT BOARD,TEENSY 4.10.STEP"
-      (offset (xyz 0 0 0))
-      (scale (xyz 1 1 1))
-      (rotate (xyz 0 0 0))
+      (offset (xyz 0 0 9.8))
+      (scale (xyz 1 1 1))
+      (rotate (xyz 0 0 0))
+    )
+    (model "${KICAD6_3DMODEL_DIR}/Connector_PinHeader_2.54mm.3dshapes/PinHeader_1x24_P2.54mm_Vertical.step"
+      (offset (xyz 29.2 7.6 9.7))
+      (scale (xyz 1 1 1))
+      (rotate (xyz 0 180 90))
+    )
+    (model "${KICAD6_3DMODEL_DIR}/Connector_PinHeader_2.54mm.3dshapes/PinHeader_1x24_P2.54mm_Vertical.step"
+      (offset (xyz 29.2 -7.6 9.7))
+      (scale (xyz 1 1 1))
+      (rotate (xyz 0 180 90))
+    )
+    (model "${KICAD6_3DMODEL_DIR}/Connector_PinSocket_2.54mm.3dshapes/PinSocket_1x24_P2.54mm_Vertical.step"
+      (offset (xyz 29.25 7.6 0.1))
+      (scale (xyz 1 1 1))
+      (rotate (xyz 0 0 90))
+    )
+    (model "${KICAD6_3DMODEL_DIR}/Connector_PinSocket_2.54mm.3dshapes/PinSocket_1x24_P2.54mm_Vertical.step"
+      (offset (xyz 29.25 -7.6 0.1))
+      (scale (xyz 1 1 1))
+      (rotate (xyz 0 0 90))
     )
   )
@@
   )
   (footprint "ESP32-Footprints:ESP82SerialTransceiver" (layer "F.Cu")
-    (at 125.705 100.155 90)
+    (at 122.14 84.68 180)
     (property "Sheetfile" "DevBoard.kicad_sch")
     (property "Sheetname" "DevBoard")
     (attr through_hole)
-    (fp_text reference "U6" (at 15.662 -0.746 180) (layer "F.SilkS") hide
-      (effects (font (size 1 1) (thickness 0.15)))
-    )
-    (fp_text value "ESP8266" (at 15.662 -11.746 180) (layer "F.SilkS")
+    (fp_text reference "U6" (at 15.662 -0.746 90) (layer "F.SilkS") hide
+      (effects (font (size 1 1) (thickness 0.15)))
+    )
+    (fp_text value "ESP8266" (at 15.662 -11.746 90) (layer "F.SilkS")
       (effects (font (size 1 1) (thickness 0.15)))
     )
@@
       ) (layer "F.SilkS") (width 0.1) (fill solid))
     (fp_line (start 1.524 -18.415) (end 1.524 -17.145) (layer "Dwgs.User") (width 0.12))
-    (pad "1" thru_hole circle locked (at 3.429 -1.524 90) (size 1.524 1.524) (drill 0.762) (layers *.Cu *.Mask)
+    (pad "1" thru_hole circle locked (at 3.429 -1.524 180) (size 1.524 1.524) (drill 0.762) (layers *.Cu *.Mask)
       (net 89 "ESP8266_UART_TX") (pinfunction "TXD") (pintype "input"))
-    (pad "2" thru_hole circle locked (at 5.969 -1.524 90) (size 1.524 1.524) (drill 0.762) (layers *.Cu *.Mask)
+    (pad "2" thru_hole circle locked (at 5.969 -1.524 180) (size 1.524 1.524) (drill 0.762) (layers *.Cu *.Mask)
       (net 85 "unconnected-(U6-Pad2)") (pinfunction "CH_PD") (pintype "input"))
-    (pad "3" thru_hole circle locked (at 8.509 -1.524 90) (size 1.524 1.524) (drill 0.762) (layers *.Cu *.Mask)
+    (pad "3" thru_hole circle locked (at 8.509 -1.524 180) (size 1.524 1.524) (drill 0.762) (layers *.Cu *.Mask)
       (net 86 "unconnected-(U6-Pad3)") (pinfunction "RST") (pintype "input"))
-    (pad "4" thru_hole circle locked (at 11.049 -1.524 90) (size 1.524 1.524) (drill 0.762) (layers *.Cu *.Mask)
+    (pad "4" thru_hole circle locked (at 11.049 -1.524 180) (size 1.524 1.524) (drill 0.762) (layers *.Cu *.Mask)
       (net 58 "+3V3") (pinfunction "VCC") (pintype "input"))
-    (pad "5" thru_hole circle locked (at 11.049 -4.064 90) (size 1.524 1.524) (drill 0.762) (layers *.Cu *.Mask)
+    (pad "5" thru_hole circle locked (at 11.049 -4.064 180) (size 1.524 1.524) (drill 0.762) (layers *.Cu *.Mask)
       (net 88 "ESP8266_UART_RX") (pinfunction "RXD") (pintype "input"))
-    (pad "6" thru_hole circle locked (at 8.509 -4.064 90) (size 1.524 1.524) (drill 0.762) (layers *.Cu *.Mask)
+    (pad "6" thru_hole circle locked (at 8.509 -4.064 180) (size 1.524 1.524) (drill 0.762) (layers *.Cu *.Mask)
       (net 87 "unconnected-(U6-Pad6)") (pinfunction "GPIO0") (pintype "input"))
-    (pad "7" thru_hole circle locked (at 5.969 -4.064 90) (size 1.524 1.524) (drill 0.762) (layers *.Cu *.Mask)
+    (pad "7" thru_hole circle locked (at 5.969 -4.064 180) (size 1.524 1.524) (drill 0.762) (layers *.Cu *.Mask)
       (net 96 "unconnected-(U6-Pad7)") (pinfunction "GPIO2") (pintype "input"))
-    (pad "8" thru_hole rect locked (at 3.429 -4.064 90) (size 1.524 1.524) (drill 0.762) (layers *.Cu *.Mask)
+    (pad "8" thru_hole rect locked (at 3.429 -4.064 180) (size 1.524 1.524) (drill 0.762) (layers *.Cu *.Mask)
       (net 45 "GND") (pinfunction "GND") (pintype "input"))
+    (model "${KICAD6_3DMODEL_DIR}/Connector_PinSocket_2.54mm.3dshapes/PinSocket_2x04_P2.54mm_Vertical.step"
+      (offset (xyz 11.05 1.5 0.1))
+      (scale (xyz 1 1 1))
+      (rotate (xyz 0 0 90))
+    )
+    (model "C:/Users/xamps/Documents/Electronics/libs/ESP-01S (ESP8266) Board Module.step"
+      (offset (xyz 0 0 11))
+      (scale (xyz 1 1 1))
+      (rotate (xyz 0 0 0))
+    )
   )
   (footprint "MiniJackConnector:MJ4435" (layer "F.Cu")
@@
       (effects (font (size 1 1) (thickness 0.15)))
     )
-    (fp_text value "TestPoint_Plated_Hole_D3.0mm" (at 0 3) (layer "F.Fab")
+    (fp_text value " " (at 0 3) (layer "F.Fab")
       (effects (font (size 1 1) (thickness 0.15)))
     )
@@
   (segment (start 140.936 59.915) (end 140.936 71.345) (width 1.016) (layer "B.Cu") (net 83))
   (segment (start 168.62 52.79) (end 166.855 51.025) (width 1.016) (layer "B.Cu") (net 83))
+  (segment (start 110.1034 84.55) (end 108.9574 85.696) (width 0.25) (layer "F.Cu") (net 88))
+  (segment (start 110.1512 88.744) (end 111.091 88.744) (width 0.25) (layer "F.Cu") (net 88))
+  (segment (start 168.62 83.27) (end 170.375 81.515) (width 0.25) (layer "F.Cu") (net 88))
+  (segment (start 155.575 84.55) (end 110.1034 84.55) (width 0.25) (layer "F.Cu") (net 88))
+  (segment (start 108.9574 85.696) (end 108.9574 87.5502) (width 0.25) (layer "F.Cu") (net 88))
+  (segment (start 170.375 80.225) (end 169.6 79.45) (width 0.25) (layer "F.Cu") (net 88))
   (segment (start 160.675 79.45) (end 155.575 84.55) (width 0.25) (layer "F.Cu") (net 88))
-  (segment (start 168.62 83.27) (end 170.375 81.515) (width 0.25) (layer "F.Cu") (net 88))
+  (segment (start 108.9574 87.5502) (end 110.1512 88.744) (width 0.25) (layer "F.Cu") (net 88))
+  (segment (start 169.6 79.45) (end 160.675 79.45) (width 0.25) (layer "F.Cu") (net 88))
   (segment (start 170.375 81.515) (end 170.375 80.225) (width 0.25) (layer "F.Cu") (net 88))
-  (segment (start 155.575 84.55) (end 126.197 84.55) (width 0.25) (layer "F.Cu") (net 88))
-  (segment (start 126.197 84.55) (end 121.641 89.106) (width 0.25) (layer "F.Cu") (net 88))
-  (segment (start 169.6 79.45) (end 160.675 79.45) (width 0.25) (layer "F.Cu") (net 88))
-  (segment (start 170.375 80.225) (end 169.6 79.45) (width 0.25) (layer "F.Cu") (net 88))
+  (segment (start 119.6762 87.1692) (end 118.711 86.204) (width 0.25) (layer "F.Cu") (net 89))
   (segment (start 155.9058 87.1692) (end 156.1298 86.9452) (width 0.254) (layer "F.Cu") (net 89))
-  (segment (start 131.432489 89.467511) (end 133.4599 87.4401) (width 0.25) (layer "F.Cu") (net 89))
+  (segment (start 133.7308 87.1692) (end 119.6762 87.1692) (width 0.25) (layer "F.Cu") (net 89))
   (segment (start 162.345 80.73) (end 168.62 80.73) (width 0.25) (layer "F.Cu") (net 89))
   (segment (start 155.9058 87.1692) (end 133.7308 87.1692) (width 0.254) (layer "F.Cu") (net 89))
   (segment (start 156.125 86.95) (end 156.1298 86.9452) (width 0.25) (layer "F.Cu") (net 89))
-  (segment (start 133.7308 87.1692) (end 133.4599 87.4401) (width 0.254) (layer "F.Cu") (net 89))
   (segment (start 156.1298 86.9452) (end 162.345 80.73) (width 0.25) (layer "F.Cu") (net 89))
-  (segment (start 124.181 96.726) (end 131.432489 89.474511) (width 0.25) (layer "F.Cu") (net 89))
-  (segment (start 131.432489 89.474511) (end 131.432489 89.467511) (width 0.25) (layer "F.Cu") (net 89))
   (segment (start 188.05 69.25) (end 188.05 67.535) (width 0.25) (layer "F.Cu") (net 90))
   (segment (start 188.05 67.535) (end 188.087 67.498) (width 0.25) (layer "F.Cu") (net 90))

Commit message: Updated and send to fab
Parts:
- moved J11 3.05 mm to (142.0, 108.0)
- moved J3 2.25 mm to (134.0, 138.3)
- moved J4 2.12 mm to (179.0, 50.9)
- moved J6 2.03 mm to (193.0, 51.0)
Routing:
- net LINE_IN_L: track 18.5 -> 22.0 mm
- net LINE_IN_R: track 20.6 -> 23.7 mm
- net USB_HOST_5V: track 157.3 -> 159.6 mm
- net HP_L: track 18.1 -> 20.2 mm
- net HP_R: track 32.4 -> 34.5 mm
- net I2C_SDA_3V3: track 119.7 -> 117.7 mm
- net HP_GND: track 38.7 -> 40.6 mm
- net I2C_SCL_3V3: track 118.5 -> 120.2 mm
- net USB_HOST_N: track 87.4 -> 88.5 mm
- net USB_HOST_P: track 87.3 -> 88.3 mm
Other:
- board text added: "CLK"
- board text added: "DT"
- board text added: "GND"
- board text added: "INT"
- board text added: "S"
- board text added: "SCL"
- board text added: "SDA"
- board text added: "SW"
- board text added: "VCC"
- board text added: "XOUT"
- board text added: "a"
- board text added: "k"

Commit message: Updated Teensy4 3d model
Parts:
- renumbered U1 to 1º
Changed lines of the file:
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@@
     (property "Sheetname" "DevBoard")
     (attr through_hole)
-    (fp_text reference "U1" (at 0 -10.16 90) (layer "F.SilkS") hide
+    (fp_text reference "1º" (at 0 -10.16 90) (layer "F.SilkS") hide
       (effects (font (size 1 1) (thickness 0.15)))
     )
@@
     (pad "67" thru_hole circle locked (at -28.48 1.27 270) (size 1.3 1.3) (drill 0.8) (layers *.Cu *.Mask)
       (net 62 "unconnected-(U1-Pad67)") (pinfunction "D+") (pintype "bidirectional"))
-    (model "C:/Users/xamps/Documents/Electronics/libs/CIRCUIT BOARD,TEENSY 4.10.STEP"
-      (offset (xyz 0 0 9.8))
-      (scale (xyz 1 1 1))
-      (rotate (xyz 0 0 0))
-    )
     (model "${KICAD6_3DMODEL_DIR}/Connector_PinHeader_2.54mm.3dshapes/PinHeader_1x24_P2.54mm_Vertical.step"
       (offset (xyz 29.2 7.6 9.7))
@@
       (rotate (xyz 0 0 90))
     )
+    (model "C:/Users/xamps/Documents/Electronics/libs/Teensy 4.1.STEP"
+      (offset (xyz 0 0 10.6))
+      (scale (xyz 1 1 1))
+      (rotate (xyz -90 0 90))
+    )
   )
